Commit message: Update robot.urdf

File: burf_robot/robot.urdf (robot description, URDF)
Before this commit: robot test_robot, 5 links, 4 joints
Links:
- link base_link: geometry collision box size=0.20 0.20 0.07; visual box size=0.20 0.20 0.07

Commit message: Sorted wheels

File: burf_robot/robot.urdf (robot description, URDF)
Before this commit: robot test_robot, 5 links, 4 joints
Links:
- removed link base_link
- added link base_frame; collision box size=0.20 0.20 0.07; visual box size=0.20 0.20 0.07
Joints:
- joint base_to_lwheel: parent base_link -> base_frame; type fixed -> continuous
- joint base_to_rwheel: parent base_link -> base_frame; type fixed -> continuous
- joint laser_joint: parent base_link -> base_frame
- joint ultrasonic_joint: parent base_link -> base_frame

Commit message: Updated

File: burf_robot/robot.urdf (robot description, URDF)
Before this commit: robot robot_model, 5 links, 4 joints
Links:
- link base_frame: geometry collision box size=0.20 0.20 0.07; visual box size=0.16 0.16 0.07
