Commit message: added collision

File: robot.urdf (robot description, URDF)
Before this commit: robot test_robot, 4 links, 3 joints
Links:
- link base_link: geometry collision box size=0.19 0.15 0.07; visual box size=0.19 0.15 0.07

Commit message: Update robot.urdf

File: robot.urdf (robot description, URDF)
Before this commit: robot test_robot, 4 links, 3 joints
Links:
- removed link laser_link
- added link laser, mass 0.00001; collision cylinder length=0.07 radius=0.02; visual box size=0.015 0.045 0.015
Joints:
- joint laser_joint: child laser_link -> laser

Commit message: Update robot.urdf

File: robot.urdf (robot description, URDF)
Before this commit: robot test_robot, 4 links, 3 joints
Links:
- added link ultrasonic; visual box size=0.02 0.02 0.02
- link laser: mass 0.00001 -> None; geometry visual cylinder length=0.01 radius=0.03
Joints:
- added joint ultrasonic_joint: type fixed, parent base_link, child ultrasonic, origin xyz=0.09 0.0 0.13 rpy=0 0 0
- joint laser_joint: origin xyz=0.1 0 0 rpy=0 0 0 -> xyz=0.0 0.0 0.125 rpy=0 0 0

Commit message: Update robot.urdf

File: robot.urdf (robot description, URDF)
Before this commit: robot robot_model, 5 links, 4 joints
Joints:
- joint base_to_lwheel: type continuous -> fixed
- joint base_to_rwheel: type continuous -> fixed

Commit message: updated wheels

File: robot.urdf (robot description, URDF)
Before this commit: robot robot_model, 5 links, 4 joints
Joints:
- joint base_to_lwheel: type fixed -> continuous
- joint base_to_rwheel: type fixed -> continuous

Commit message: Adding settings for vex tank

File: robot.urdf (robot description, URDF)
Before this commit: robot robot_model, 5 links, 4 joints
Links:
- link base_frame: geometry collision box size=1.10 0.90 0.15; visual box size=1.10 0.80 0.15
- link laser: geometry visual cylinder length=0.03 radius=0.08
- link lwheel: geometry visual cylinder length=0.03 radius=0.105
- link rwheel: geometry visual cylinder length=0.03 radius=0.105
Joints:
- joint base_to_lwheel: origin xyz=0 0.085 0.07 rpy=1.5708 0 0 -> xyz=0 0.42 0.06 rpy=1.5708 0 0
- joint base_to_rwheel: origin xyz=0 -0.085 0.07 rpy=-1.5708 0 0 -> xyz=0 -0.42 0.06 rpy=-1.5708 0 0
- joint laser_joint: origin xyz=0.0 0.0 0.125 rpy=0 0 0 -> xyz=-0.5 0.0 0.80 rpy=0 0 0
